Commit message: rplidar urdf updates

File: genbu_description/urdf/robot.urdf.xacro (robot description, xacro)
@@ -3,3 +3,4 @@
   <xacro:include filename="$(find create_description)/urdf/create_2.urdf.xacro" />
   <xacro:include filename="$(find genbu_description)/urdf/rplidar.urdf.xacro" />
+  <xacro:rplidar parent="base_link" xyz="0.042 -0.042 0.0720" rpy="0 0 -1.571" />
 </robot>

File: genbu_description/urdf/rplidar.urdf.xacro (robot description, xacro)
@@ -2,5 +2,6 @@
 <robot xmlns:xacro="http://www.ros.org/wiki/xacro" name="rplidar">
   <xacro:macro name="rplidar" params="parent:=base_link xyz:='0 0 0' rpy:='0 0 0'">
-    <link name="rplidar_link">
+    <!-- Base of the RPLIDAR (below the center of the motor) -->
+    <link name="rplidar_base_link">
       <visual>
         <geometry>
@@ -9,8 +10,16 @@
       </visual>
     </link>
-    <joint name="rplidar_joint" type="fixed">
+    <joint name="rplidar_base_joint" type="fixed">
       <parent link="${parent}"/>
-      <child link="rplidar_link"/>
+      <child link="rplidar_base_link"/>
       <origin xyz="${xyz}" rpy="${rpy}"/>
+    </joint>
+    <!-- Laser link (position of the laser sensor ) -->
+    <link name="rplidar_laser_link">
+    </link>
+    <joint name="rplidar_laser_joint" type="fixed">
+      <parent link="rplidar_base_link"/>
+      <child link="rplidar_laser_link"/>
+      <origin xyz="-0.0455 0 0.042" rpy="0 0 0"/>
     </joint>
   </xacro:macro>
