Commit message: Serve robot mesh assets for Foxglove
Co-authored-by: nnarain <8395093+nnarain@users.noreply.github.com>

File: genbu_description/urdf/robot.urdf.xacro (robot description, xacro)
@@ -1,6 +1,8 @@
 <?xml version="1.0" ?>
 <robot name="genbu" xmlns:xacro="http://ros.org/wiki/xacro">
+  <xacro:arg name="mesh_base_url" default="package://genbu_description/meshes"/>
   <xacro:include filename="$(find create_description)/urdf/create_2.urdf.xacro" />
   <xacro:include filename="$(find genbu_description)/urdf/ydlidar.urdf.xacro" />
-  <xacro:ydlidar parent="base_link" xyz="0.042 -0.042 0.0720" rpy="0 0 -1.571" />
+  <xacro:ydlidar parent="base_link" xyz="0.042 -0.042 0.0720" rpy="0 0 -1.571"
+    mesh_base_url="$(arg mesh_base_url)" />
 </robot>

File: genbu_description/urdf/rplidar.urdf.xacro (robot description, xacro)
@@ -1,6 +1,6 @@
 <?xml version="1.0"?>
 <robot xmlns:xacro="http://www.ros.org/wiki/xacro" name="rplidar">
-  <xacro:macro name="rplidar" params="parent:=base_link xyz:='0 0 0' rpy:='0 0 0'">
-  <xacro:property name="mesh_file" value="package://genbu_description/meshes/rplidar_a1m8.dae"/>
+  <xacro:macro name="rplidar" params="parent:=base_link xyz:='0 0 0' rpy:='0 0 0' mesh_base_url:='package://genbu_description/meshes'">
+  <xacro:property name="mesh_file" value="${mesh_base_url}/rplidar_a1m8.dae"/>
     <!-- Base of the RPLIDAR (below the center of the motor) -->
     <link name="rplidar_base_link">

File: genbu_description/urdf/ydlidar.urdf.xacro (robot description, xacro)
@@ -1,7 +1,7 @@
 <?xml version="1.0"?>
 <robot xmlns:xacro="http://www.ros.org/wiki/xacro" name="ydlidar">
-  <xacro:macro name="ydlidar" params="parent:=base_link xyz:='0 0 0' rpy:='0 0 0'">
+  <xacro:macro name="ydlidar" params="parent:=base_link xyz:='0 0 0' rpy:='0 0 0' mesh_base_url:='package://genbu_description/meshes'">
   <!-- Mesh file for the RPLIDAR, used for visualization in RViz/Simulation. -->
-  <xacro:property name="mesh_file" value="package://genbu_description/meshes/rplidar_a1m8.dae"/>
+  <xacro:property name="mesh_file" value="${mesh_base_url}/rplidar_a1m8.dae"/>
     <!-- Base of the YDLidar (physical mount). No mesh available for this sensor. -->
     <link name="ydlidar_base_link">

Commit message: Remove standalone Foxglove mesh server
Co-authored-by: nnarain <8395093+nnarain@users.noreply.github.com>

File: genbu_description/urdf/robot.urdf.xacro (robot description, xacro)
@@ -1,8 +1,6 @@
 <?xml version="1.0" ?>
 <robot name="genbu" xmlns:xacro="http://ros.org/wiki/xacro">
-  <xacro:arg name="mesh_base_url" default="package://genbu_description/meshes"/>
   <xacro:include filename="$(find create_description)/urdf/create_2.urdf.xacro" />
   <xacro:include filename="$(find genbu_description)/urdf/ydlidar.urdf.xacro" />
-  <xacro:ydlidar parent="base_link" xyz="0.042 -0.042 0.0720" rpy="0 0 -1.571"
-    mesh_base_url="$(arg mesh_base_url)" />
+  <xacro:ydlidar parent="base_link" xyz="0.042 -0.042 0.0720" rpy="0 0 -1.571" />
 </robot>

File: genbu_description/urdf/rplidar.urdf.xacro (robot description, xacro)
@@ -1,6 +1,6 @@
 <?xml version="1.0"?>
 <robot xmlns:xacro="http://www.ros.org/wiki/xacro" name="rplidar">
-  <xacro:macro name="rplidar" params="parent:=base_link xyz:='0 0 0' rpy:='0 0 0' mesh_base_url:='package://genbu_description/meshes'">
-  <xacro:property name="mesh_file" value="${mesh_base_url}/rplidar_a1m8.dae"/>
+  <xacro:macro name="rplidar" params="parent:=base_link xyz:='0 0 0' rpy:='0 0 0'">
+  <xacro:property name="mesh_file" value="package://genbu_description/meshes/rplidar_a1m8.dae"/>
     <!-- Base of the RPLIDAR (below the center of the motor) -->
     <link name="rplidar_base_link">

File: genbu_description/urdf/ydlidar.urdf.xacro (robot description, xacro)
@@ -1,7 +1,7 @@
 <?xml version="1.0"?>
 <robot xmlns:xacro="http://www.ros.org/wiki/xacro" name="ydlidar">
-  <xacro:macro name="ydlidar" params="parent:=base_link xyz:='0 0 0' rpy:='0 0 0' mesh_base_url:='package://genbu_description/meshes'">
+  <xacro:macro name="ydlidar" params="parent:=base_link xyz:='0 0 0' rpy:='0 0 0'">
   <!-- Mesh file for the RPLIDAR, used for visualization in RViz/Simulation. -->
-  <xacro:property name="mesh_file" value="${mesh_base_url}/rplidar_a1m8.dae"/>
+  <xacro:property name="mesh_file" value="package://genbu_description/meshes/rplidar_a1m8.dae"/>
     <!-- Base of the YDLidar (physical mount). No mesh available for this sensor. -->
     <link name="ydlidar_base_link">
