Commit message: Resolves #6. Initial simulation bringup

File: genbu_description/urdf/rplidar.urdf.xacro (robot description, xacro)
@@ -2,9 +2,10 @@
 <robot xmlns:xacro="http://www.ros.org/wiki/xacro" name="rplidar">
   <xacro:macro name="rplidar" params="parent:=base_link xyz:='0 0 0' rpy:='0 0 0'">
+  <xacro:property name="mesh_file" value="file://$(find genbu_description)/meshes/rplidar_a1m8.dae"/>
     <!-- Base of the RPLIDAR (below the center of the motor) -->
     <link name="rplidar_base_link">
       <visual>
         <geometry>
-          <mesh filename="package://genbu_description/meshes/rplidar_a1m8.dae" scale="1 1 1"/>
+          <mesh filename="${mesh_file}" scale="1 1 1"/>
         </geometry>
       </visual>
