Commit message: Use package URIs for lidar meshes
Co-authored-by: nnarain <8395093+nnarain@users.noreply.github.com>

File: genbu_description/urdf/rplidar.urdf.xacro (robot description, xacro)
@@ -2,5 +2,5 @@
 <robot xmlns:xacro="http://www.ros.org/wiki/xacro" name="rplidar">
   <xacro:macro name="rplidar" params="parent:=base_link xyz:='0 0 0' rpy:='0 0 0'">
-  <xacro:property name="mesh_file" value="file://$(find genbu_description)/meshes/rplidar_a1m8.dae"/>
+  <xacro:property name="mesh_file" value="package://genbu_description/meshes/rplidar_a1m8.dae"/>
     <!-- Base of the RPLIDAR (below the center of the motor) -->
     <link name="rplidar_base_link">

File: genbu_description/urdf/ydlidar.urdf.xacro (robot description, xacro)
@@ -3,5 +3,5 @@
   <xacro:macro name="ydlidar" params="parent:=base_link xyz:='0 0 0' rpy:='0 0 0'">
   <!-- Mesh file for the RPLIDAR, used for visualization in RViz/Simulation. -->
-  <xacro:property name="mesh_file" value="file://$(find genbu_description)/meshes/rplidar_a1m8.dae"/>
+  <xacro:property name="mesh_file" value="package://genbu_description/meshes/rplidar_a1m8.dae"/>
     <!-- Base of the YDLidar (physical mount). No mesh available for this sensor. -->
     <link name="ydlidar_base_link">
