Commit message: fix lidar position

File: genbu_description/urdf/ydlidar.urdf.xacro (robot description, xacro)
@@ -2,6 +2,13 @@
 <robot xmlns:xacro="http://www.ros.org/wiki/xacro" name="ydlidar">
   <xacro:macro name="ydlidar" params="parent:=base_link xyz:='0 0 0' rpy:='0 0 0'">
+  <!-- Mesh file for the RPLIDAR, used for visualization in RViz/Simulation. -->
+  <xacro:property name="mesh_file" value="file://$(find genbu_description)/meshes/rplidar_a1m8.dae"/>
     <!-- Base of the YDLidar (physical mount). No mesh available for this sensor. -->
     <link name="ydlidar_base_link">
+      <visual>
+        <geometry>
+          <mesh filename="${mesh_file}" scale="1 1 1"/>
+        </geometry>
+      </visual>
     </link>
     <joint name="ydlidar_base_joint" type="fixed">
@@ -17,5 +24,5 @@
       <parent link="ydlidar_base_link"/>
       <child link="laser"/>
-      <origin xyz="0 0 0" rpy="0 0 0"/>
+      <origin xyz="0 0 0.042" rpy="0 0 0"/>
     </joint>
     <!-- Gazebo lidar sensor at the laser link -->

Commit message: fix lidar orientation

File: genbu_description/urdf/ydlidar.urdf.xacro (robot description, xacro)
@@ -24,5 +24,5 @@
       <parent link="ydlidar_base_link"/>
       <child link="laser"/>
-      <origin xyz="0 0 0.042" rpy="0 0 0"/>
+      <origin xyz="0 0 0.042" rpy="0 0 -1.57"/>
     </joint>
     <!-- Gazebo lidar sensor at the laser link -->

Commit message: actually fix the lidar orientation

File: genbu_description/urdf/ydlidar.urdf.xacro (robot description, xacro)
@@ -24,5 +24,5 @@
       <parent link="ydlidar_base_link"/>
       <child link="laser"/>
-      <origin xyz="0 0 0.042" rpy="0 0 -1.57"/>
+      <origin xyz="0 0 0.042" rpy="0 0 1.5708"/>
     </joint>
     <!-- Gazebo lidar sensor at the laser link -->

Commit message: nav settings

File: genbu_description/urdf/ydlidar.urdf.xacro (robot description, xacro)
@@ -24,5 +24,5 @@
       <parent link="ydlidar_base_link"/>
       <child link="laser"/>
-      <origin xyz="0 0 0.042" rpy="0 0 1.5708"/>
+      <origin xyz="0 0 0.042" rpy="0 0 0"/>
     </joint>
     <!-- Gazebo lidar sensor at the laser link -->

Commit message: fix lidar yaw

File: genbu_description/urdf/ydlidar.urdf.xacro (robot description, xacro)
@@ -24,5 +24,5 @@
       <parent link="ydlidar_base_link"/>
       <child link="laser"/>
-      <origin xyz="0 0 0.042" rpy="0 0 0"/>
+      <origin xyz="0 0 0.042" rpy="0 0 1.57079632679"/>
     </joint>
     <!-- Gazebo lidar sensor at the laser link -->
